File: boards/controller/eyevend-controller/eyevend-controller.kicad_sch (KiCad schematic)
At the start: 8 parts, among them J2 Conn_01x03, J3 Conn_01x03, J4 Micro_SD_Card, U1 Pico, U2 _DAC8411

Commit message: updated board
Parts:
- removed U2: _DAC8411, symbol JFHDAC:_DAC8411
- added C2, C3: 0.1u, Capacitor_SMD:C_0402_1005Metric, symbol Device:C
- added C4: 1u, Capacitor_SMD:C_0402_1005Metric, symbol Device:C
- added J1: pwr_in, symbol Connector_Generic:Conn_01x02
- added J5, J7: Conn_01x15, Connector_PinHeader_2.54mm:PinHeader_1x15_P2.54mm_Vertical, symbol Connector_Generic:Conn_01x15
- added R2: 10k, Resistor_SMD:R_0402_1005Metric, symbol Device:R
- added SW1: SW_Push, symbol Switch:SW_Push
- added U2: DAC8411, Package_TO_SOT_SMD:Texas_R-PDSO-G6, symbol JFHDAC:DAC8411
- added U3: PAM8302AAD, symbol Amplifier_Audio:PAM8302AAD
- C1: value C -> 10n; footprint (none) -> Capacitor_SMD:C_0402_1005Metric
- J2: value Conn_01x03 -> sig
- J3: value Conn_01x03 -> swd
- R1: value R -> 10k; footprint (none) -> Resistor_SMD:R_0402_1005Metric
Connections:
- net mSD_CS: now reaches J4.2 (DAT3/CD)
- net mSD_CS: now also U1.2 (GPIO1)
- net SPI_COPI: now reaches J4.3 (CMD)
- net SPI_COPI: now also U1.5 (GPIO3), U2.3 (DIN)
- net +3.3V: now reaches J4.4 (VDD)
- net +3.3V: now also J2.1 (Pin_1), U1.36 (3V3), C2.1, C3.1, C4.1, J5.1 (Pin_1), J5.15 (Pin_15), J7.1 (Pin_1), J7.15 (Pin_15)
- net SPI_CLK: now reaches J4.5 (CLK)
- net SPI_CLK: now also U1.4 (GPIO2), U2.2 (SCK)
- net GND: now reaches J4.6 (VSS)
- net GND: now also J3.2 (Pin_2), J4.9 (SHIELD), U1.13 (GND), U1.18 (GND), U1.23 (GND), U1.28 (GND), U1.3 (GND), U1.38 (GND), U1.42 (GND), U1.8 (GND), J1.2 (Pin_2), J5.13 (Pin_13), J5.5 (Pin_5), J5.9 (Pin_9), J7.13 (Pin_13), J7.5 (Pin_5), J7.9 (Pin_9), SW1.2
- net SPI_CIPO: now reaches J4.7 (DAT0)
- net SPI_CIPO: now also U1.6 (GPIO4)
- net SWDIO: now reaches J3.1 (Pin_1)
- net SWDIO: now also U1.43 (SWDIO)
- net SWCLK: now reaches J3.3 (Pin_3)
- net SWCLK: now also U1.41 (SWCLK)
- net at LS1.1: now also U3.5 (OUT+)
- net at LS1.2: now also U3.8 (OUT-)
- net at R1.1: now also C1.1, U3.3 (IN+)
- net at R1.2: now also U2.6 (VOUT)
- net DAC_CS: now reaches U1.1 (GPIO0)
- net DAC_CS: now also U2.1 (SYNC)
- net GP7: now reaches U1.10 (GPIO7)
- net GP7: now also J5.4 (Pin_4)
- net GP8: now reaches U1.11 (GPIO8)
- net GP8: now also J5.6 (Pin_6)
- net GP9: now reaches U1.12 (GPIO9)
- net GP9: now also J5.7 (Pin_7)
- net GP10: now reaches U1.14 (GPIO10)
- net GP10: now also J5.8 (Pin_8)
- net GP11: now reaches U1.15 (GPIO11)
- net GP11: now also J5.10 (Pin_10)
- net GP12: now reaches U1.16 (GPIO12)
- net GP12: now also J5.11 (Pin_11)
- net GP13: now reaches U1.17 (GPIO13)
- net GP13: now also J5.12 (Pin_12)
- net GP14: now reaches U1.19 (GPIO14)
- net GP14: now also J7.2 (Pin_2)
- net GP15: now reaches U1.20 (GPIO15)
- net GP15: now also J7.3 (Pin_3)
- net GP16: now reaches U1.21 (GPIO16)
- net GP16: now also J7.4 (Pin_4)
- net GP17: now reaches U1.22 (GPIO17)
- net GP17: now also J7.6 (Pin_6)
- net GP18: now reaches U1.24 (GPIO18)
- net GP18: now also J7.7 (Pin_7)
- net GP19: now reaches U1.25 (GPIO19)
- net GP19: now also J7.8 (Pin_8)
- net GP20: now reaches U1.26 (GPIO20)
- net GP20: now also J7.10 (Pin_10)
- net GP21: now reaches U1.27 (GPIO21)
- net GP21: now also J7.11 (Pin_11)
- net GP22: now reaches U1.29 (GPIO22)
- net GP22: now also J7.12 (Pin_12)
- net at U1.30 (RUN): now also SW1.1
- net GP26: now reaches U1.31 (GPIO26_ADC0)
- net GP26: now also J7.14 (Pin_14)
- net GP27: now reaches U1.32 (GPIO27_ADC1)
- net GP27: now also J5.14 (Pin_14)
- net GNDA: now reaches U1.33 (AGND)
- net GNDA: now also C1.2, J2.3 (Pin_3), C2.2, C3.2, C4.2, U2.5 (GND), U3.4 (IN-), U3.7 (GND)
- net SIG: now reaches U1.34 (GPIO28_ADC2)
- net SIG: now also J2.2 (Pin_2)
- net +5V: now reaches U1.39 (VSYS)
- net +5V: now also J1.1 (Pin_1)
- net GP5: now reaches U1.7 (GPIO5)
- net GP5: now also J5.2 (Pin_2)
- net GP6: now reaches U1.9 (GPIO6)
- net GP6: now also J5.3 (Pin_3)
- new net: R2.1, U3.1 (~{SD})
- new net VDDA: R2.2, U2.4 (VDDA)
- no-connect marks 0 -> 5
Other:
- note added: "Audio"
- note added: "GPIO"
- note added: "Pico"
- note added: "Ports"
- note added: "Storage"
- note removed: "buffer stage/ speaker amp stage?"
- note removed: "how to drive the speaker?"
- company: (none) -> JHorwitzDesign
- title: (none) -> EyeVend Controller Board
- moved on the sheet: C1, J4, LS1, R1, U1

Commit message: board finished, need to order still
Parts:
- removed J1: pwr_in, symbol Connector_Generic:Conn_01x02
- removed J4: Micro_SD_Card, symbol Connector:Micro_SD_Card
- added C5: 1u, Capacitor_SMD:C_0402_1005Metric, symbol Device:C
- added J1: Barrel_Jack_Switch, JFH=Connector_DC_Jack:DC-0440-2.5A-2.5, symbol Connector:Barrel_Jack_Switch
- added J4: pwr_utilL, Connector_JST:JST_PH_S2B-PH-K_1x02_P2.00mm_Horizontal, symbol Connector_Generic:Conn_01x02
- added J6: Micro_SD_Card_Det1, JFHsd:GT-TF003-H0185-02, symbol Connector:Micro_SD_Card_Det1
- added J8: pwr_utilR, Connector_JST:JST_PH_S2B-PH-K_1x02_P2.00mm_Horizontal, symbol Connector_Generic:Conn_01x02
- added J9: sig, Connector_JST:JST_PH_S3B-PH-K_1x03_P2.00mm_Horizontal, symbol Connector_Generic:Conn_01x03
- added U4: GND_STARPOINT, JFH=Connector_DC_Jack:gndstarpoint, symbol JFHAnalog:GND_STARPOINT
- J2: footprint (none) -> Connector_JST:JST_PH_S3B-PH-K_1x03_P2.00mm_Horizontal
- J3: footprint (none) -> Connector_PinHeader_2.54mm:PinHeader_1x03_P2.54mm_Vertical
- LS1: footprint (none) -> Connector_JST:JST_PH_B2B-PH-K_1x02_P2.00mm_Vertical
- SW1: footprint (none) -> Buttons:PTS636 6.0x3.5 Button
- U1: footprint RPi_Pico:RPi_Pico_SMD_TH -> MCU_RaspberryPi_and_Boards:RPi_Pico_SMD_TH
- U3: footprint (none) -> Package_SO:MSOP-8_3x3mm_P0.65mm
Connections:
- net VDDA is gone; now on net +3.3V: R2.2, U2.4 (VDDA)
- net +3.3V: now also U3.6 (VDD), C5.1, J6.4 (VDD), J9.1 (Pin_1)
- net +5V: now also J1.1, J4.1 (Pin_1), J8.1 (Pin_1)
- net GND: now also C3.2, J5.2 (Pin_2), J1.2, J4.2 (Pin_2), J6.10 (SHIELD), J6.6 (VSS), U4.2 (gnd)
- net GNDA: now also C5.2, J8.2 (Pin_2), J9.3 (Pin_3), U4.1 (gnda); no longer C3.2
- net GP14: now also J5.14 (Pin_14); no longer J7.2 (Pin_2)
- net GP15: now also J7.14 (Pin_14); no longer J7.3 (Pin_3)
- net GP16: now also J7.2 (Pin_2); no longer J7.4 (Pin_4)
- net GP17: now also J7.3 (Pin_3); no longer J7.6 (Pin_6)
- net GP18: now also J7.4 (Pin_4); no longer J7.7 (Pin_7)
- net GP19: now also J7.6 (Pin_6); no longer J7.8 (Pin_8)
- net GP20: now also J7.7 (Pin_7); no longer J7.10 (Pin_10)
- net GP21: now also J7.8 (Pin_8); no longer J7.11 (Pin_11)
- net GP22: now also J7.10 (Pin_10); no longer J7.12 (Pin_12)
- net GP26: now also J7.11 (Pin_11); no longer J7.14 (Pin_14)
- net GP27: now also J7.12 (Pin_12); no longer J5.14 (Pin_14)
- net SIG: now also J9.2 (Pin_2)
- net SPI_CIPO: now also J6.7 (DAT0)
- net SPI_CLK: now also J6.5 (CLK)
- net SPI_COPI: now also J6.3 (CMD)
- net mSD_CS: now also J6.2 (DAT3/CD)
- net GP5 renamed SD_CD
- net SD_CD: now also J6.9 (DET); no longer J5.2 (Pin_2)
- no-connect marks 5 -> 6
Other:
- note added: "jst ph"

Commit message: added mounting holes
Parts:
- added H1, H2, H3, H4: MountingHole_Pad, MountingHole:MountingHole_2.2mm_M2_ISO7380, symbol Mechanical:MountingHole_Pad
Connections:
- net GND: now also H1.1, H2.1, H3.1
- net GNDA: now also H4.1
Changed lines of the file:
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@@
+    (stroke (width 0) (type default))
+  )
+  (wire (pts (xy 144.78 179.07) (xy 144.78 177.8))
     (stroke (width 0) (type default))
   )
@@
     (stroke (width 0) (type default))
   )
+  (wire (pts (xy 120.65 167.64) (xy 120.65 166.37))
+    (stroke (width 0) (type default))
+  )
   (wire (pts (xy 129.54 113.03) (xy 138.43 113.03))
     (stroke (width 0) (type default))
@@
     (stroke (width 0) (type default))
   )
+  (wire (pts (xy 144.78 167.64) (xy 144.78 166.37))
+    (stroke (width 0) (type default))
+  )
   (wire (pts (xy 93.98 158.75) (xy 93.98 160.02))
     (stroke (width 0) (type default))
@@
   )
   (wire (pts (xy 262.89 129.54) (xy 262.89 128.27))
+    (stroke (width 0) (type default))
+  )
+  (wire (pts (xy 120.65 179.07) (xy 120.65 177.8))
     (stroke (width 0) (type default))
   )
@@
     )
   )
+  (symbol (lib_id "power:GND") (at 120.65 179.07 0) (unit 1)
+    (in_bom yes) (on_board yes) (dnp no)
+    (property "Reference" "#PWR053" (at 120.65 185.42 0)
+      (effects (font (size 1.27 1.27)) hide)
+    )
+    (property "Value" "GND" (at 124.46 180.34 0)
+      (effects (font (size 1.27 1.27)))
+    )
+    (property "Footprint" "" (at 120.65 179.07 0)
+      (effects (font (size 1.27 1.27)) hide)
+    )
+    (property "Datasheet" "" (at 120.65 179.07 0)
+      (effects (font (size 1.27 1.27)) hide)
+    )
+    (pin "1")
+    (instances
+      (project "eyevend-controller"
+        (path "/5f1e92c2-955c-4939-a9ba-2ed8574a5c2a"
+          (reference "#PWR053") (unit 1)
+        )
+      )
+    )
+  )
   (symbol (lib_id "JFHDAC:DAC8411") (at 175.26 49.53 0) (unit 1)
     (in_bom yes) (on_board yes) (dnp no)
@@
         (path "/5f1e92c2-955c-4939-a9ba-2ed8574a5c2a"
           (reference "#PWR018") (unit 1)
+        )
+      )
+    )
+  )
+  (symbol (lib_id "Mechanical:MountingHole_Pad") (at 144.78 175.26 0) (unit 1)
+    (in_bom yes) (on_board yes) (dnp no) (fields_autoplaced)
+    (property "Reference" "H4" (at 147.32 172.72 0)
+      (effects (font (size 1.27 1.27)) (justify left))
+    )
+    (property "Value" "MountingHole_Pad" (at 147.32 175.26 0)
+      (effects (font (size 1.27 1.27)) (justify left))
+    )
+    (property "Footprint" "MountingHole:MountingHole_2.2mm_M2_ISO7380" (at 144.78 175.26 0)
+      (effects (font (size 1.27 1.27)) hide)
+    )
+    (property "Datasheet" "~" (at 144.78 175.26 0)
+      (effects (font (size 1.27 1.27)) hide)
+    )
+    (pin "1")
+    (instances
+      (project "eyevend-controller"
+        (path "/5f1e92c2-955c-4939-a9ba-2ed8574a5c2a"
+          (reference "H4") (unit 1)
         )
       )
@@
     )
   )
+  (symbol (lib_id "power:GND") (at 120.65 167.64 0) (unit 1)
+    (in_bom yes) (on_board yes) (dnp no)
+    (property "Reference" "#PWR051" (at 120.65 173.99 0)
+      (effects (font (size 1.27 1.27)) hide)
+    )
+    (property "Value" "GND" (at 124.46 168.91 0)
+      (effects (font (size 1.27 1.27)))
+    )
+    (property "Footprint" "" (at 120.65 167.64 0)
+      (effects (font (size 1.27 1.27)) hide)
+    )
+    (property "Datasheet" "" (at 120.65 167.64 0)
+      (effects (font (size 1.27 1.27)) hide)
+    )
+    (pin "1")
+    (instances
+      (project "eyevend-controller"
+        (path "/5f1e92c2-955c-4939-a9ba-2ed8574a5c2a"
+          (reference "#PWR051") (unit 1)
+        )
+      )
+    )
+  )
   (symbol (lib_id "power:GNDA") (at 91.44 63.5 0) (unit 1)
     (in_bom yes) (on_board yes) (dnp no)
@@
         (path "/5f1e92c2-955c-4939-a9ba-2ed8574a5c2a"
           (reference "C4") (unit 1)
+        )
+      )
+    )
+  )
+  (symbol (lib_id "power:GNDA") (at 144.78 179.07 0) (unit 1)
+    (in_bom yes) (on_board yes) (dnp no)
+    (property "Reference" "#PWR054" (at 144.78 185.42 0)
+      (effects (font (size 1.27 1.27)) hide)
+    )
+    (property "Value" "GNDA" (at 148.59 180.34 0)
+      (effects (font (size 1.27 1.27)))
+    )
+    (property "Footprint" "" (at 144.78 179.07 0)
+      (effects (font (size 1.27 1.27)) hide)
+    )
+    (property "Datasheet" "" (at 144.78 179.07 0)
+      (effects (font (size 1.27 1.27)) hide)
+    )
+    (pin "1")
+    (instances
+      (project "eyevend-controller"
+        (path "/5f1e92c2-955c-4939-a9ba-2ed8574a5c2a"
+          (reference "#PWR054") (unit 1)
         )
       )
@@
         (path "/5f1e92c2-955c-4939-a9ba-2ed8574a5c2a"
           (reference "U3") (unit 1)
+        )
+      )
+    )
+  )
+  (symbol (lib_id "Mechanical:MountingHole_Pad") (at 144.78 163.83 0) (unit 1)
+    (in_bom yes) (on_board yes) (dnp no) (fields_autoplaced)
+    (property "Reference" "H2" (at 147.32 161.29 0)
+      (effects (font (size 1.27 1.27)) (justify left))
+    )
+    (property "Value" "MountingHole_Pad" (at 147.32 163.83 0)
+      (effects (font (size 1.27 1.27)) (justify left))
+    )
+    (property "Footprint" "MountingHole:MountingHole_2.2mm_M2_ISO7380" (at 144.78 163.83 0)
+      (effects (font (size 1.27 1.27)) hide)
+    )
+    (property "Datasheet" "~" (at 144.78 163.83 0)
+      (effects (font (size 1.27 1.27)) hide)
+    )
+    (pin "1")
+    (instances
+      (project "eyevend-controller"
+        (path "/5f1e92c2-955c-4939-a9ba-2ed8574a5c2a"
+          (reference "H2") (unit 1)
         )
       )
@@
     )
   )
+  (symbol (lib_id "Mechanical:MountingHole_Pad") (at 120.65 175.26 0) (unit 1)
+    (in_bom yes) (on_board yes) (dnp no) (fields_autoplaced)
+    (property "Reference" "H3" (at 123.19 172.72 0)
+      (effects (font (size 1.27 1.27)) (justify left))
+    )
+    (property "Value" "MountingHole_Pad" (at 123.19 175.26 0)
+      (effects (font (size 1.27 1.27)) (justify left))
+    )
+    (property "Footprint" "MountingHole:MountingHole_2.2mm_M2_ISO7380" (at 120.65 175.26 0)
+      (effects (font (size 1.27 1.27)) hide)
+    )
+    (property "Datasheet" "~" (at 120.65 175.26 0)
+      (effects (font (size 1.27 1.27)) hide)
+    )
+    (pin "1")
+    (instances
+      (project "eyevend-controller"
+        (path "/5f1e92c2-955c-4939-a9ba-2ed8574a5c2a"
+          (reference "H3") (unit 1)
+        )
+      )
+    )
+  )
   (symbol (lib_id "Connector_Generic:Conn_01x03") (at 213.36 144.78 0) (unit 1)
     (in_bom yes) (on_board yes) (dnp no)
@@
     )
   )
+  (symbol (lib_id "Mechanical:MountingHole_Pad") (at 120.65 163.83 0) (unit 1)
+    (in_bom yes) (on_board yes) (dnp no) (fields_autoplaced)
+    (property "Reference" "H1" (at 123.19 161.29 0)
+      (effects (font (size 1.27 1.27)) (justify left))
+    )
+    (property "Value" "MountingHole_Pad" (at 123.19 163.83 0)
+      (effects (font (size 1.27 1.27)) (justify left))
+    )
+    (property "Footprint" "MountingHole:MountingHole_2.2mm_M2_ISO7380" (at 120.65 163.83 0)
+      (effects (font (size 1.27 1.27)) hide)
+    )
+    (property "Datasheet" "~" (at 120.65 163.83 0)
+      (effects (font (size 1.27 1.27)) hide)
+    )
+    (pin "1")
+    (instances
+      (project "eyevend-controller"
+        (path "/5f1e92c2-955c-4939-a9ba-2ed8574a5c2a"
+          (reference "H1") (unit 1)
+        )
+      )
+    )
+  )
   (symbol (lib_id "power:+3.3V") (at 204.47 140.97 0) (unit 1)
     (in_bom yes) (on_board yes) (dnp no)
@@
         )
       )
+    )
+  )
+  (symbol (lib_id "power:GND") (at 144.78 167.64 0) (unit 1)
+    (in_bom yes) (on_board yes) (dnp no)
+    (property "Reference" "#PWR052" (at 144.78 173.99 0)
+      (effects (font (size 1.27 1.27)) hide)
+    )
+    (property "Value" "GND" (at 148.59 168.91 0)
+      (effects (font (size 1.27 1.27)))
+    )
+    (property "Footprint" "" (at 144.78 167.64 0)
+      (effects (font (size 1.27 1.27)) hide)
+    )
+    (property "Datasheet" "" (at 144.78 167.64 0)
+      (effects (font (size 1.27 1.27)) hide)
+    )
+    (pin "1")
+    (instances
+      (project "eyevend-controller"
+        (path "/5f1e92c2-955c-4939-a9ba-2ed8574a5c2a"
+          (reference "#PWR052") (unit 1)
+        )
+      )
